File: 2-4GHz-Remote/Receiver.sch (KiCad schematic (older format))
At the start: 4 parts

Commit message: updated schematic
Connections:
- net Sheet5BC7EAF8/L_IN: now reaches J?.1 (L_IN)
- net Sheet5BC7EAF8/N_IN: now reaches J?.2 (N_IN)
- net Sheet5BC7EAF8/N_OUT: now reaches J?.3 (N_OUT)
- net Sheet5BC7EAF8/L_OUT: now reaches J?.4 (L_OUT)
Changed lines of the file:
@@
 F0 "Sheet5BC7EAF8" 50
 F1 "Monstrum.sch" 50
+F2 "L_IN" I L 4550 5600 50
+F3 "N_IN" I L 4550 6400 50
+F4 "N_OUT" I R 5950 6400 50
+F5 "L_OUT" I R 5950 5600 50
 $EndSheet
+Wire Wire Line
+	4550 5600 4300 5600
+Wire Wire Line
+	4300 5600 4300 5100
+Wire Wire Line
+	4300 5100 4950 5100
+Wire Wire Line
+	4950 5100 4950 4650
+Wire Wire Line
+	5100 4650 5100 5000
+Wire Wire Line
+	5100 5000 4200 5000
+Wire Wire Line
+	4200 5000 4200 6400
+Wire Wire Line
+	4200 6400 4550 6400
+Wire Wire Line
+	5950 5600 6200 5600
+Wire Wire Line
+	6200 5600 6200 5050
+Wire Wire Line
+	6200 5050 5550 5050
+Wire Wire Line
+	5550 5050 5550 4650
+Wire Wire Line
+	5950 6400 6300 6400
+Wire Wire Line
+	6300 6400 6300 4950
+Wire Wire Line
+	6300 4950 5400 4950
+Wire Wire Line
+	5400 4950 5400 4650
 $EndSCHEMATC

Commit message: SChematic updates
Parts:
- J?: symbol Remote_parts:4PIN_PLUG -> 2-4GHz-Remote-rescue:4PIN_PLUG-Remote_parts
- J?: symbol Remote_parts:4PIN_SOCKET -> 2-4GHz-Remote-rescue:4PIN_SOCKET-Remote_parts
Changed lines of the file:
@@
 	7800 3650 9600 3650
 $Comp
-L Remote_parts:4PIN_PLUG J?
+L 2-4GHz-Remote-rescue:4PIN_PLUG-Remote_parts J?
 U 1 1 5BC61BD1
 P 5250 3650
+AR Path="/5BC61BD1" Ref="J?"  Part="1"
+AR Path="/5BC4CC0A/5BC61BD1" Ref="J?"  Part="1"
 F 0 "J?" H 5878 3276 50  0000 L CNN
 F 1 "4PIN_PLUG" H 5878 3185 50  0000 L CNN
@@
 $EndComp
 $Comp
-L Remote_parts:4PIN_SOCKET J?
+L 2-4GHz-Remote-rescue:4PIN_SOCKET-Remote_parts J?
 U 1 1 5BC7300A
 P 5250 2950
